Commit message: Add wheels to Eduard offroad model.

File: model/urdf/eduard.urdf (robot description, URDF)
Before this commit: robot eduard, 1 links, 0 joints
Links:
- added link wheel_front_left; visual mesh filename=package://edu_robot_control/model/mesh/offroad-wheel-eduard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
- added link wheel_front_right; visual mesh filename=package://edu_robot_control/model/mesh/offroad-wheel-eduard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
- added link wheel_rear_left; visual mesh filename=package://edu_robot_control/model/mesh/offroad-wheel-eduard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
- added link wheel_rear_right; visual mesh filename=package://edu_robot_control/model/mesh/offroad-wheel-eduard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
Joints:
- added joint base_to_wheel_front_left: type fixed, parent base_link, child wheel_front_left
- added joint base_to_wheel_front_right: type fixed, parent base_link, child wheel_front_right
- added joint base_to_wheel_rear_left: type fixed, parent base_link, child wheel_rear_left
- added joint base_to_wheel_rear_right: type fixed, parent base_link, child wheel_rear_right

Commit message: Fix joints for Eduard robot.

File: model/urdf/eduard.urdf (robot description, URDF)
Before this commit: robot eduard, 5 links, 4 joints
Joints:
- joint base_to_wheel_front_left: axis (none) -> 0 0 1; origin (none) -> xyz=0.125 0.163 0.02 rpy=1.570796327 0 0; type fixed -> continuous
- joint base_to_wheel_front_right: axis (none) -> 0 0 1; origin (none) -> xyz=0.125 -0.163 0.02 rpy=-1.570796327 0 0; type fixed -> continuous
- joint base_to_wheel_rear_left: axis (none) -> 0 0 1; origin (none) -> xyz=-0.125 0.163 0.02 rpy=1.570796327 0 0; type fixed -> continuous
- joint base_to_wheel_rear_right: axis (none) -> 0 0 1; origin (none) -> xyz=-0.125 -0.163 0.02 rpy=-1.570796327 0 0; type fixed -> continuous

Commit message: Switch wheel rotation in SDF file.

File: model/urdf/eduard.urdf (robot description, URDF)
Before this commit: robot eduard, 5 links, 4 joints
Joints:
- joint base_to_wheel_front_left: origin xyz=0.125 0.163 0.02 rpy=1.570796327 0 0 -> xyz=0.125 0.163 0.02 rpy=-1.570796327 0 0
- joint base_to_wheel_front_right: origin xyz=0.125 -0.163 0.02 rpy=-1.570796327 0 0 -> xyz=0.125 -0.163 0.02 rpy=1.570796327 0 0
- joint base_to_wheel_rear_left: origin xyz=-0.125 0.163 0.02 rpy=1.570796327 0 0 -> xyz=-0.125 0.163 0.02 rpy=-1.570796327 0 0
- joint base_to_wheel_rear_right: origin xyz=-0.125 -0.163 0.02 rpy=-1.570796327 0 0 -> xyz=-0.125 -0.163 0.02 rpy=1.570796327 0 0

Commit message: Switch to humble: next steps.

File: model/urdf/eduard.urdf (robot description, URDF)
Before this commit: robot eduard, 5 links, 4 joints
Links:
- removed link base_link
- removed link wheel_front_left
- removed link wheel_front_right
- removed link wheel_rear_left
- removed link wheel_rear_right
- added link $(arg robot_name)/base_link; visual mesh filename=package://edu_robot_control/model/mesh/eduard-chassis.dae
- added link $(arg robot_name)/wheel_front_left; visual mesh filename=package://edu_robot_control/model/mesh/offroad-wheel-eduard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
- added link $(arg robot_name)/wheel_front_right; visual mesh filename=package://edu_robot_control/model/mesh/offroad-wheel-eduard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
- added link $(arg robot_name)/wheel_rear_left; visual mesh filename=package://edu_robot_control/model/mesh/offroad-wheel-eduard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
- added link $(arg robot_name)/wheel_rear_right; visual mesh filename=package://edu_robot_control/model/mesh/offroad-wheel-eduard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
Joints:
- removed joint base_to_wheel_front_left
- removed joint base_to_wheel_front_right
- removed joint base_to_wheel_rear_left
- removed joint base_to_wheel_rear_right
- added joint $(arg robot_name)/base_to_wheel_front_left: type continuous, parent $(arg robot_name)/base_link, child $(arg robot_name)/wheel_front_left, origin xyz=0.125 0.163 0.02 rpy=-1.570796327 0 0, axis 0 0 1
- added joint $(arg robot_name)/base_to_wheel_front_right: type continuous, parent $(arg robot_name)/base_link, child $(arg robot_name)/wheel_front_right, origin xyz=0.125 -0.163 0.02 rpy=1.570796327 0 0, axis 0 0 1
- added joint $(arg robot_name)/base_to_wheel_rear_left: type continuous, parent $(arg robot_name)/base_link, child $(arg robot_name)/wheel_rear_left, origin xyz=-0.125 0.163 0.02 rpy=-1.570796327 0 0, axis 0 0 1
- added joint $(arg robot_name)/base_to_wheel_rear_right: type continuous, parent $(arg robot_name)/base_link, child $(arg robot_name)/wheel_rear_right, origin xyz=-0.125 -0.163 0.02 rpy=1.570796327 0 0, axis 0 0 1

Commit message: Fix wrong rotation direction in RVIZ model description. Add docker instructions to readme file.

File: model/urdf/eduard.urdf (robot description, URDF)
Before this commit: robot $(arg robot_name), 5 links, 4 joints
Joints:
- joint $(arg robot_name)/base_to_wheel_front_left: origin xyz=0.125 0.163 0.02 rpy=-1.570796327 0 0 -> xyz=0.125 0.163 0.02 rpy=1.570796327 0 0
- joint $(arg robot_name)/base_to_wheel_front_right: origin xyz=0.125 -0.163 0.02 rpy=1.570796327 0 0 -> xyz=0.125 -0.163 0.02 rpy=-1.570796327 0 0
- joint $(arg robot_name)/base_to_wheel_rear_left: origin xyz=-0.125 0.163 0.02 rpy=-1.570796327 0 0 -> xyz=-0.125 0.163 0.02 rpy=1.570796327 0 0
- joint $(arg robot_name)/base_to_wheel_rear_right: origin xyz=-0.125 -0.163 0.02 rpy=1.570796327 0 0 -> xyz=-0.125 -0.163 0.02 rpy=-1.570796327 0 0

Commit message: Add wheel type to robot description.

File: model/urdf/eduard.urdf (robot description, URDF)
Before this commit: robot $(arg robot_name), 5 links, 4 joints
Links:
- link $(arg robot_name)/base_link: geometry 
- link $(arg robot_name)/wheel_front_left: geometry visual {http://ros.org/wiki/xacro}if value=${'offroad' in '$(arg wheel_type)'}
- link $(arg robot_name)/wheel_front_right: geometry visual {http://ros.org/wiki/xacro}if value=${'offroad' in '$(arg wheel_type)'}
- link $(arg robot_name)/wheel_rear_left: geometry visual {http://ros.org/wiki/xacro}if value=${'offroad' in '$(arg wheel_type)'}
- link $(arg robot_name)/wheel_rear_right: geometry visual {http://ros.org/wiki/xacro}if value=${'offroad' in '$(arg wheel_type)'}
